File: lokalizator.sch (EAGLE design)
At the start: 19 parts, among them IC1 ATMEGA328PROUND, X1 1268-120, X2 1268-120, X3 1297-25, X4 1297-25

Commit message: Add files via upload
Parts:
- U$2: value GSM-MODEM-SIM900A -> GSM-MODULE-G510
Changed lines of the file:
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@@
 <part name="U$4" library="diy-modules2" deviceset="LIGHT-SENSOR-BH1750" device="" value="ACCELEROMETER SENSOR"/>
 <part name="U$3" library="diy-modules2" deviceset="GPS-RECEIVER-NEO6M" device=""/>
-<part name="U$2" library="diy-modules2" deviceset="GSM-MODEM-SIM900A" device=""/>
+<part name="U$2" library="diy-modules2" deviceset="GSM-MODEM-SIM900A" device="" value="GSM-MODULE-G510"/>
 <part name="X3" library="con-commcon" library_urn="urn:adsk.eagle:library:134" deviceset="1297-25" device="" package3d_urn="urn:adsk.eagle:package:6281/1"/>
 <part name="X4" library="con-commcon" library_urn="urn:adsk.eagle:library:134" deviceset="1297-25" device="" package3d_urn="urn:adsk.eagle:package:6281/1"/>
