File: Hardware/Lokalizator Płytka Uniwersalna/lokalizator_płytka_uniwersalna.sch (EAGLE design)
At the start: 18 parts, among them IC1 ATMEGA328PROUND

Commit message: Add files via upload
Parts:
- removed JP1, JP2, JP4: (no value), adafruit:PINHD-1X1
- added X1, X2: 1268-120, con-commcon:1268-120
- added X3, X4: 1297-25, con-commcon:1297-25
Connections:
- new net N$1: R2.1, SW1.P$2, X1A.14, X1B.14, X1C.14, X1D.14
- new net N$10: IC1.(PCI0/ICP/CLKO)PB0, X1A.30, X1B.30, X1C.30, X1D.30
- new net N$19: IC1.(PCI1/OC1A/OC1S)PB1, X2A.30, X2B.30, X2C.30, X2D.30
- new net N$20: IC1.(PCI2/SS/OC1B)PB2, X2A.29, X2B.29, X2C.29, X2D.29
- new net N$23: IC1.(PCI21/T1/OC0B)PD5, X1A.27, X1B.27, X1C.27, X1D.27
- new net N$24: IC1.(PCI8/ADC0)PC0, X2A.22, X2B.22, X2C.22, X2D.22
- new net N$25: IC1.(PCI19/INT1/OC2B)PD3, X1A.21, X1B.21, X1C.21, X1D.21
- new net N$26: IC1.(PCI12/ADC4/SDA)PC4, U$4.SDA, X2A.13, X2A.18, X2B.13, X2B.18, X2C.13, X2C.18, X2D.13, X2D.18
- new net N$27: IC1.(PCI20/XCK/T0)PD4, X1A.22, X1B.22, X1C.22, X1D.22
- new net N$28: X1A.15, X1B.15, X1C.15, X1D.15
- new net N$29: X1A.13, X1B.13, X1C.13, X1D.13
- new net N$30: X1A.12, X1B.12, X1C.12, X1D.12
- new net N$31: X1A.11, X1B.11, X1C.11, X1D.11
- new net N$32: X1A.10, X1B.10, X1C.10, X1D.10
- new net N$33: X1A.9, X1B.9, X1C.9, X1D.9
- new net N$37: X1A.5, X1B.5, X1C.5, X1D.5
- new net N$38: X1A.4, X1B.4, X1C.4, X1D.4
- new net N$39: X1A.3, X1B.3, X1C.3, X1D.3
- new net N$40: X1A.2, X1B.2, X1C.2, X1D.2
- new net N$41: X1A.1, X1B.1, X1C.1, X1D.1
- new net N$42: X2A.16, X2B.16, X2C.16, X2D.16
- new net N$43: X2A.15, X2B.15, X2C.15, X2D.15
- new net N$44: X2A.14, X2B.14, X2C.14, X2D.14
- new net N$48: X2A.10, X2B.10, X2C.10, X2D.10
- new net N$50: X2A.8, X2B.8, X2C.8, X2D.8
- new net N$51: X2A.7, X2B.7, X2C.7, X2D.7
- new net N$52: X2A.6, X2B.6, X2C.6, X2D.6
- new net N$53: X2A.5, X2B.5, X2C.5, X2D.5
- new net N$54: X2A.4, X2B.4, X2C.4, X2D.4
- new net N$55: X2A.3, X2B.3, X2C.3, X2D.3
- new net N$57: X2A.1, X2B.1, X2C.1, X2D.1
- new net N$7: C4.1, IC1.PB7(XTAL2/TOSC2/PCI7), Q1.1, X1A.26, X1B.26, X1C.26, X1D.26
- net GND: now also X1A.24, X1A.7, X1B.24, X1B.7, X1C.24, X1C.7, X1D.24, X1D.7, X2A.11, X2A.23, X2B.11, X2B.23, X2C.11, X2C.23, X2D.11, X2D.23, X3B.1, X3B.10, X3B.11, X3B.12, X3B.13, X3B.14, X3B.15, X3B.16, X3B.17, X3B.18, X3B.19, X3B.2, X3B.20, X3B.21, X3B.22, X3B.23, X3B.24, X3B.25, X3B.3, X3B.4, X3B.5, X3B.6, X3B.7, X3B.8, X3B.9, X4B.1, X4B.10, X4B.11, X4B.12, X4B.13, X4B.14, X4B.15, X4B.16, X4B.17, X4B.18, X4B.19, X4B.2, X4B.20, X4B.21, X4B.22, X4B.23, X4B.24, X4B.25, X4B.3, X4B.4, X4B.5, X4B.6, X4B.7, X4B.8, X4B.9; no longer JP4.1
- net N$11: now also IC1.(PCI13/ADC5/SCL)PC5, U$4.SCL, X2A.12, X2A.17, X2B.12, X2B.17, X2C.12, X2C.17, X2D.12, X2D.17; no longer C4.1, IC1.PB7(XTAL2/TOSC2/PCI7), Q1.1
- net N$12: now also X1A.16, X1B.16, X1C.16, X1D.16; no longer IC1.(PCI12/ADC4/SDA)PC4, U$4.SDA
- net N$13: now also X1A.20, X1A.6, X1B.20, X1B.6, X1C.20, X1C.6, X1D.20, X1D.6
- net N$14: now also X2A.21, X2B.21, X2C.21, X2D.21
- net N$15: now also X1A.18, X1B.18, X1C.18, X1D.18
- net N$16: now also X1A.19, X1B.19, X1C.19, X1D.19
- net N$17: now also X2A.20, X2B.20, X2C.20, X2D.20
- net N$18: now also X2A.19, X2B.19, X2C.19, X2D.19
- net N$2: now also X1A.17, X1B.17, X1C.17, X1D.17
- net N$21: now also IC1.(PCI23/AIN1)PD7, X1A.29, X1B.29, X1C.29, X1D.29; no longer IC1.(PCI13/ADC5/SCL)PC5, U$4.SCL
- net N$22: now also IC1.(PCI22/AIN0OC0A)PD6, X1A.28, X1B.28, X1C.28, X1D.28; no longer R2.1, SW1.P$2
- net N$3: now also X2A.24, X2B.24, X2C.24, X2D.24
- net N$5: now also X2A.26, X2B.26, X2C.26, X2D.26
- net N$6: now also X1A.25, X1B.25, X1C.25, X1D.25
- net N$8: now also X2A.27, X2B.27, X2C.27, X2D.27
- net N$9: now also X2A.28, X2B.28, X2C.28, X2D.28
- net VCC: now also X1A.23, X1A.8, X1B.23, X1B.8, X1C.23, X1C.8, X1D.23, X1D.8, X2A.2, X2A.25, X2A.9, X2B.2, X2B.25, X2B.9, X2C.2, X2C.25, X2C.9, X2D.2, X2D.25, X2D.9, X3A.1, X3A.10, X3A.11, X3A.12, X3A.13, X3A.14, X3A.15, X3A.16, X3A.17, X3A.18, X3A.19, X3A.2, X3A.20, X3A.21, X3A.22, X3A.23, X3A.24, X3A.25, X3A.3, X3A.4, X3A.5, X3A.6, X3A.7, X3A.8, X3A.9, X4A.1, X4A.10, X4A.11, X4A.12, X4A.13, X4A.14, X4A.15, X4A.16, X4A.17, X4A.18, X4A.19, X4A.2, X4A.20, X4A.21, X4A.22, X4A.23, X4A.24, X4A.25, X4A.3, X4A.4, X4A.5, X4A.6, X4A.7, X4A.8, X4A.9; no longer JP1.1, JP2.1
Other:
- moved on the sheet: C1, C2, C4, C5, C6, JP10, JP13, JP3, Q1, R2, SW1, U$2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
